File: Board/SAP-1.brd (EAGLE design)
At the start: 100 x 100 mm, 227 parts

Commit message: added CPU status register
Parts:
- added ALU:C1, ALU:C2, ALU:C3, ALU:C4, ALU:C5, ALU:C6, ALU:C7, SR:C1: 100n, rcl:C050-024X044
- added ALU:IC6: 74LS02N, 74xx-us:DIL14
- added ALU:IC7: 74ALS08N, 74xx-us:DIL14
- added ID:FI: (no value), led:LED3MM
- added ID:R17: 10k, rcl:0204/7
- added SR:IC2: 74LS173N, 74xx-us:DIL16
- added SR:LED1: RED, led:LED3MM
- added SR:LED2: GREEN, led:LED3MM
- ID:R16: value 10k -> 220
- moved ID:R16 58.0 mm to (-16.0, 205.0)
- moved RB:LED1 1.27 mm to (94.6, 34.3)
- moved RB:LED2 1.27 mm to (90.2, 34.3)
- moved RB:LED3 1.27 mm to (85.7, 34.3)
- moved RB:LED4 1.27 mm to (81.3, 34.3)
- moved RB:LED5 1.27 mm to (76.8, 34.3)
- moved RB:LED6 1.27 mm to (72.4, 34.3)
- moved RB:LED7 1.27 mm to (67.9, 34.3)
- moved RB:LED8 1.27 mm to (63.5, 34.3)
- renumbered ID:LED1 to ID:HLT, ID:LED10 to ID:SU, ID:LED11 to ID:BI, ID:LED12 to ID:OI, ID:LED13 to ID:CE, ID:LED14 to ID:CO, ID:LED15 to ID:JP, ID:LED16 to ID:T0, ID:LED17 to ID:T1, ID:LED18 to ID:T2, ID:LED19 to ID:T3, ID:LED2 to ID:MI, ID:LED20 to ID:T4, ID:LED3 to ID:RO, ID:LED4 to ID:RI, ID:LED5 to ID:IO, ID:LED6 to ID:II, ID:LED7 to ID:AO, ID:LED8 to ID:AI, ID:LED9 to ID:EO
Connections:
- removed net ALU:N$9: ALU:LED1.K, ALU:LED2.K, ALU:LED3.K, ALU:LED4.K, ALU:LED5.K, ALU:LED6.K, ALU:LED7.K, ALU:LED8.K
- removed net RA:N$4: RA:LED1.K, RA:LED2.K, RA:LED3.K, RA:LED4.K, RA:LED5.K, RA:LED6.K, RA:LED7.K, RA:LED8.K
- removed net RB:N$16: RB:LED1.K, RB:LED2.K, RB:LED3.K, RB:LED4.K, RB:LED5.K, RB:LED6.K, RB:LED7.K, RB:LED8.K
- new net !FI: ID:IC4.10, SR:IC2.10, SR:IC2.9
- new net ALU:N$2: ALU:IC6.1, ALU:IC7.1
- new net ALU:N$3: ALU:IC6.4, ALU:IC7.2
- new net ALU:N$4: ALU:IC6.10, ALU:IC7.4
- new net ALU:N$5: ALU:IC6.13, ALU:IC7.5
- new net ALU:N$6: ALU:IC7.3, ALU:IC7.9
- new net ALU:N$7: ALU:IC7.10, ALU:IC7.6
- new net CF: ID:IC1.23, ID:IC2.23, SR:IC2.3, SR:LED2.A
- new net ID:N$30: ID:IC2.17, ID:IC4.11
- new net ID:N$31: ID:FI.K, ID:R16.2
- new net ID:N$32: ID:FI.A
- new net SR:GND: SR:C1.2, SR:IC2.1, SR:IC2.2, SR:IC2.8, SR:LED1.K, SR:LED2.K
- new net SR:VCC: SR:C1.1, SR:IC2.16
- new net ZF: ID:IC1.22, ID:IC2.22, SR:IC2.4, SR:LED1.A
- new net ZR: ALU:IC7.8, SR:IC2.13
- net !AI: no longer ID:AI.A
- net !AO: no longer ID:AO.A
- net !BI: no longer ID:BI.A
- net !CO: no longer ID:CO.A
- net !EO: no longer ID:EO.A
- net !II: no longer ID:II.A
- net !IO: no longer ID:IO.A
- net !JP: no longer ID:JP.A
- net !MI: no longer ID:MI.A
- net !RO: no longer ID:RO.A
- net ALU:GND: now also ALU:C1.2, ALU:C2.2, ALU:C3.2, ALU:C4.2, ALU:C5.2, ALU:C6.2, ALU:C7.2, ALU:IC6.7, ALU:IC7.7, ALU:LED1.K, ALU:LED2.K, ALU:LED3.K, ALU:LED4.K, ALU:LED5.K, ALU:LED6.K, ALU:LED7.K, ALU:LED8.K
- net ALU:S1: now also ALU:IC6.2
- net ALU:S2: now also ALU:IC6.3
- net ALU:S3: now also ALU:IC6.5
- net ALU:S4: now also ALU:IC6.6
- net ALU:S5: now also ALU:IC6.8
- net ALU:S6: now also ALU:IC6.9
- net ALU:S7: now also ALU:IC6.11
- net ALU:S8: now also ALU:IC6.12
- net ALU:VCC: now also ALU:C1.1, ALU:C2.1, ALU:C3.1, ALU:C4.1, ALU:C5.1, ALU:C6.1, ALU:C7.1, ALU:IC6.14, ALU:IC7.14
- net CLR: now also SR:IC2.15
- net CY: now also SR:IC2.14
- net ID:GND: now also ID:R17.1; no longer ID:IC1.22, ID:IC1.23, ID:IC2.1, ID:IC2.22, ID:IC2.23
- net ID:N$16: now also ID:R17.2; no longer ID:R16.2
- net ID:N$20: now also ID:MI.A
- net ID:N$21: now also ID:RO.A
- net ID:N$22: now also ID:IO.A
- net ID:N$23: now also ID:II.A
- net ID:N$24: now also ID:AO.A
- net ID:N$25: now also ID:AI.A
- net ID:N$26: now also ID:EO.A
- net ID:N$27: now also ID:BI.A
- net ID:N$28: now also ID:CO.A
- net ID:N$29: now also ID:JP.A
- net ID:VCC: now also ID:IC2.1
- net N$22: now also SR:IC2.7
- net RA:GND: now also RA:LED1.K, RA:LED2.K, RA:LED3.K, RA:LED4.K, RA:LED5.K, RA:LED6.K, RA:LED7.K, RA:LED8.K
- net RB:GND: now also RB:LED1.K, RB:LED2.K, RB:LED3.K, RB:LED4.K, RB:LED5.K, RB:LED6.K, RB:LED7.K, RB:LED8.K
Routing:
- net N$13: track 33.9 -> 32.5 mm
- net N$14: track 30.6 -> 29.3 mm
- net N$12: track 25.0 -> 23.9 mm
- net N$11: track 53.3 -> 52.3 mm
- net N$15: track 32.2 -> 31.6 mm
- net N$9: track 58.9 -> 58.4 mm
- net N$16: track 33.8 -> 33.3 mm
- net N$10: track 55.9 -> 55.4 mm

Commit message: added current limiting resistors
Parts:
- removed CLK:R7: 1k, rcl:0204/7
- added ALU:R1, ALU:R2, ALU:R3, ALU:R4, ALU:R5, ALU:R6, ALU:R7, ALU:R8, CLK:R11, ID:R21, ID:R22, ID:R23, ID:R24, ID:R25, IR:R1, IR:R2, IR:R3, IR:R4, IR:R5, IR:R6, IR:R7, IR:R8, MAR:R1, MAR:R2, MAR:R3, MAR:R4, PC:R1, PC:R2, PC:R3, PC:R4, RA:R1, RA:R2, RA:R3, RA:R4, RA:R5, RA:R6, RA:R7, RA:R8, RAM:R1, RAM:R2, RAM:R3, RAM:R4, RAM:R5, RAM:R6, RAM:R7, RAM:R8, RB:R1, RB:R2, RB:R3, RB:R4, RB:R5, RB:R6, RB:R7, RB:R8, SR:R1, SR:R2: 220, rcl:0204/7
- CLK:R2: device SparkFun-Electromechanical:ALPS_POT_KIT -> rcl:RTRIM64W
- R10, R11, R12, R13, R14, R15, R16, R9: value 470 -> 220
Connections:
- new net ALU:N$10: ALU:LED6.K, ALU:R6.2
- new net ALU:N$11: ALU:LED5.K, ALU:R5.2
- new net ALU:N$12: ALU:LED4.K, ALU:R4.2
- new net ALU:N$13: ALU:LED3.K, ALU:R3.2
- new net ALU:N$14: ALU:LED2.K, ALU:R2.2
- new net ALU:N$15: ALU:LED1.K, ALU:R1.2
- new net ALU:N$8: ALU:LED8.K, ALU:R8.2
- new net ALU:N$9: ALU:LED7.K, ALU:R7.2
- new net CLK:N$4: CLK:LED1.K, CLK:R11.2
- new net ID:N$33: ID:R23.2, ID:T2.K
- new net ID:N$34: ID:R25.2, ID:T4.K
- new net ID:N$35: ID:R24.2, ID:T3.K
- new net ID:N$36: ID:R22.2, ID:T1.K
- new net ID:N$37: ID:R21.2, ID:T0.K
- new net IR:N$1: IR:LED8.K, IR:R8.2
- new net IR:N$2: IR:LED7.K, IR:R7.2
- new net IR:N$3: IR:LED6.K, IR:R6.2
- new net IR:N$5: IR:LED5.K, IR:R5.2
- new net IR:N$6: IR:LED4.K, IR:R4.2
- new net IR:N$7: IR:LED3.K, IR:R3.2
- new net IR:N$8: IR:LED2.K, IR:R2.2
- new net IR:N$9: IR:LED1.K, IR:R1.2
- new net MAR:N$10: MAR:LED1.K, MAR:R1.2
- new net MAR:N$2: MAR:LED4.K, MAR:R4.2
- new net MAR:N$4: MAR:LED3.K, MAR:R3.2
- new net MAR:N$8: MAR:LED2.K, MAR:R2.2
- new net PC:N$1: PC:LED4.K, PC:R4.2
- new net PC:N$2: PC:LED3.K, PC:R3.2
- new net PC:N$3: PC:LED2.K, PC:R2.2
- new net PC:N$4: PC:LED1.K, PC:R1.2
- new net RA:N$1: RA:LED1.K, RA:R1.2
- new net RA:N$2: RA:LED2.K, RA:R2.2
- new net RA:N$3: RA:LED3.K, RA:R3.2
- new net RA:N$4: RA:LED4.K, RA:R4.2
- new net RA:N$5: RA:LED5.K, RA:R5.2
- new net RA:N$6: RA:LED6.K, RA:R6.2
- new net RA:N$7: RA:LED7.K, RA:R7.2
- new net RA:N$8: RA:LED8.K, RA:R8.2
- new net RAM:N$10: RAM:LED7.K, RAM:R7.2
- new net RAM:N$11: RAM:LED6.K, RAM:R6.2
- new net RAM:N$12: RAM:LED5.K, RAM:R5.2
- new net RAM:N$13: RAM:LED4.K, RAM:R4.2
- new net RAM:N$14: RAM:LED3.K, RAM:R3.2
- new net RAM:N$15: RAM:LED2.K, RAM:R2.2
- new net RAM:N$16: RAM:LED1.K, RAM:R1.2
- new net RAM:N$9: RAM:LED8.K, RAM:R8.2
- new net RB:N$1: RB:LED8.K, RB:R8.2
- new net RB:N$2: RB:LED7.K, RB:R7.2
- new net RB:N$3: RB:LED6.K, RB:R6.2
- new net RB:N$4: RB:LED5.K, RB:R5.2
- new net RB:N$5: RB:LED4.K, RB:R4.2
- new net RB:N$6: RB:LED3.K, RB:R3.2
- new net RB:N$7: RB:LED2.K, RB:R2.2
- new net RB:N$8: RB:LED1.K, RB:R1.2
- new net SR:N$1: SR:LED1.K, SR:R2.2
- new net SR:N$2: SR:LED2.K, SR:R1.2
- net ALU:GND: now also ALU:R1.1, ALU:R2.1, ALU:R3.1, ALU:R4.1, ALU:R5.1, ALU:R6.1, ALU:R7.1, ALU:R8.1; no longer ALU:LED1.K, ALU:LED2.K, ALU:LED3.K, ALU:LED4.K, ALU:LED5.K, ALU:LED6.K, ALU:LED7.K, ALU:LED8.K
- net CLK:GND: now also CLK:R11.1; no longer CLK:LED1.K, CLK:R7.1
- net CLK:N$1: now also CLK:R2.1, CLK:R2.2; no longer CLK:R2.P$2, CLK:R2.P$3
- net CLK:N$3: now also CLK:R2.3; no longer CLK:R2.P$1
- net HLT: no longer CLK:R7.2
- net ID:GND: now also ID:R21.1, ID:R22.1, ID:R23.1, ID:R24.1, ID:R25.1; no longer ID:T0.K, ID:T1.K, ID:T2.K, ID:T3.K, ID:T4.K
- net IR:N$4: now also IR:R1.1, IR:R2.1, IR:R3.1, IR:R4.1, IR:R5.1, IR:R6.1, IR:R7.1, IR:R8.1; no longer IR:LED1.K, IR:LED2.K, IR:LED3.K, IR:LED4.K, IR:LED5.K, IR:LED6.K, IR:LED7.K, IR:LED8.K
- net MAR:GND: now also MAR:R1.1, MAR:R2.1, MAR:R3.1, MAR:R4.1; no longer MAR:LED1.K, MAR:LED2.K, MAR:LED3.K, MAR:LED4.K
- net PC:GND: now also PC:R1.1, PC:R2.1, PC:R3.1, PC:R4.1; no longer PC:LED1.K, PC:LED2.K, PC:LED3.K, PC:LED4.K
- net RA:GND: now also RA:R1.1, RA:R2.1, RA:R3.1, RA:R4.1, RA:R5.1, RA:R6.1, RA:R7.1, RA:R8.1; no longer RA:LED1.K, RA:LED2.K, RA:LED3.K, RA:LED4.K, RA:LED5.K, RA:LED6.K, RA:LED7.K, RA:LED8.K
- net RAM:GND: now also RAM:R1.1, RAM:R2.1, RAM:R3.1, RAM:R4.1, RAM:R5.1, RAM:R6.1, RAM:R7.1, RAM:R8.1; no longer RAM:LED1.K, RAM:LED2.K, RAM:LED3.K, RAM:LED4.K, RAM:LED5.K, RAM:LED6.K, RAM:LED7.K, RAM:LED8.K
- net RB:GND: now also RB:R1.1, RB:R2.1, RB:R3.1, RB:R4.1, RB:R5.1, RB:R6.1, RB:R7.1, RB:R8.1; no longer RB:LED1.K, RB:LED2.K, RB:LED3.K, RB:LED4.K, RB:LED5.K, RB:LED6.K, RB:LED7.K, RB:LED8.K
- net SR:GND: now also SR:R1.1, SR:R2.1; no longer SR:LED1.K, SR:LED2.K

Commit message: added mouser part numbers
Parts:
- ALU:IC7, CLK:IC6, OUT:IC2: value 74ALS08N -> 74LS08N
- ALU:LED1, ALU:LED2, ALU:LED3, ALU:LED5, ALU:LED6, ALU:LED7, ALU:LED8, ID:AI, ID:AO, ID:BI, ID:CE, ID:CO, ID:EO, ID:FI, ID:HLT, ID:II, ID:IO, ID:JP, ID:MI, ID:OI, ID:RI, ID:RO, ID:SU, LED1, LED2, LED3, LED4, LED5, LED6, LED7, LED8: value (none) -> RED
- CLK:C1: device rcl:E2,5-5 -> rcl:E2,5-7
- CLK:S2: value (none) -> Source Select
- ID:IC3, ID:IC4: value 74ALS04N -> 74LS04N
- ID:IC7, RAM:IC9: value 74ALS00N -> 74LS00N
- ID:T0, ID:T1, ID:T2, ID:T3, ID:T4: value (none) -> GREEN
- IR:LED1, IR:LED2, IR:LED3, IR:LED4, MAR:LED1, MAR:LED2, MAR:LED3, MAR:LED4, RAM:LED1, RAM:LED2, RAM:LED3, RAM:LED4: value BLUE -> RED
- IR:LED5, IR:LED6, IR:LED7, IR:LED8: value YELLOW -> BLUE
- MAR:S3: value (none) -> Program / Write
- OUT:IC3: value 74273N -> 74LS273N
- RAM:IC1, RAM:IC2: value 74LS189LSN -> 74LS189N
- RAM:LED5, RAM:LED6, RAM:LED7, RAM:LED8: value YELLOW -> RED
- SR:LED2: value GREEN -> RED
- moved ID:IC4 1428.0 mm to (-8.89, 461.0)
- moved ID:IC3 1333.6 mm to (-8.89, 449.6)
- moved CLK:C1 1.27 mm to (16.0, 56.5)
