File: Board/SAP-1.brd (EAGLE design)
At the start: 100 x 100 mm, 297 parts

Commit message: added BOM
Parts:
- added C1: (no value), rcl:E3,5-8
- added C6: 100n, rcl:C050-024X044
- added U$1: DC-JACK, Parts:POWER_JACK_PTH
Connections:
- new net VCC: C1.+, C6.1, U$1.PWR
- net GND: now also C1.-, C6.2, U$1.GND, U$1.GNDBREAK
Changed lines of the file:
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@@
 <layer number="112" name="tSilk" color="7" fill="1" visible="yes" active="yes"/>
 <layer number="113" name="IDFDebug" color="7" fill="1" visible="yes" active="yes"/>
+<layer number="114" name="Badge_Outline" color="7" fill="1" visible="yes" active="yes"/>
+<layer number="115" name="ReferenceISLANDS" color="7" fill="1" visible="yes" active="yes"/>
 <layer number="116" name="Patch_BOT" color="9" fill="4" visible="yes" active="yes"/>
+<layer number="117" name="BACKMAAT1" color="7" fill="1" visible="yes" active="yes"/>
 <layer number="118" name="Rect_Pads" color="7" fill="1" visible="yes" active="yes"/>
+<layer number="119" name="KAP_TEKEN" color="7" fill="1" visible="yes" active="yes"/>
+<layer number="120" name="KAP_MAAT1" color="7" fill="1" visible="yes" active="yes"/>
 <layer number="121" name="_tsilk" color="7" fill="1" visible="yes" active="yes"/>
 <layer number="122" name="_bsilk" color="7" fill="1" visible="yes" active="yes"/>
@@
 <layer number="128" name="_bValues" color="7" fill="1" visible="yes" active="yes"/>
 <layer number="129" name="Mask" color="7" fill="1" visible="yes" active="yes"/>
+<layer number="130" name="SMDSTROOK" color="7" fill="1" visible="yes" active="yes"/>
 <layer number="131" name="tAdjust" color="7" fill="1" visible="yes" active="yes"/>
 <layer number="132" name="bAdjust" color="7" fill="1" visible="yes" active="yes"/>
+<layer number="133" name="bottom_silk" color="7" fill="1" visible="yes" active="yes"/>
+<layer number="134" name="silk_top" color="7" fill="1" visible="no" active="no"/>
+<layer number="135" name="silk_bottom" color="7" fill="1" visible="no" active="no"/>
+<layer number="136" name="silktop" color="7" fill="1" visible="yes" active="yes"/>
+<layer number="137" name="silkbottom" color="7" fill="1" visible="yes" active="yes"/>
 <layer number="144" name="Drill_legend" color="7" fill="1" visible="yes" active="yes"/>
+<layer number="145" name="DrillLegend_01-16" color="7" fill="1" visible="yes" active="yes"/>
+<layer number="146" name="DrillLegend_01-20" color="7" fill="1" visible="yes" active="yes"/>
 <layer number="150" name="Notes" color="7" fill="1" visible="yes" active="yes"/>
 <layer number="151" name="HeatSink" color="7" fill="1" visible="yes" active="yes"/>
@@
 <layer number="230" name="230bmp" color="7" fill="1" visible="yes" active="yes"/>
 <layer number="231" name="231bmp" color="7" fill="1" visible="yes" active="yes"/>
+<layer number="232" name="Eagle3D_PG2" color="7" fill="1" visible="yes" active="yes"/>
+<layer number="233" name="Eagle3D_PG3" color="7" fill="1" visible="yes" active="yes"/>
 <layer number="248" name="Housing" color="7" fill="1" visible="yes" active="yes"/>
 <layer number="249" name="Edge" color="7" fill="1" visible="yes" active="yes"/>
@@
 <elements>
 <element name="CLK:C1" library="rcl" library_urn="urn:adsk.eagle:library:334" package="E2,5-7" package3d_urn="urn:adsk.eagle:package:23345/1" value="1u" x="15.955" y="56.465" smashed="yes">
-<attribute name="CONRAD" value="445639" x="15.955" y="56.465" size="1.778" layer="27" display="off"/>
 <attribute name="MOUSER" value="710-860021373002" x="15.955" y="56.465" size="1.778" layer="27" display="off"/>
 <attribute name="NAME" x="18.368" y="57.735" size="1.27" layer="25" ratio="10"/>
@@
 <attribute name="VALUE" x="-15.621" y="460.375" size="1.27" layer="27" ratio="10"/>
 </element>
+<element name="C1" library="rcl" library_urn="urn:adsk.eagle:library:334" package="E3,5-8" package3d_urn="urn:adsk.eagle:package:23360/2" value="" x="-16.51" y="-1182.37" smashed="yes">
+<attribute name="MOUSER" value="710-860040674004" x="-16.51" y="-1182.37" size="1.778" layer="27" display="off"/>
+<attribute name="NAME" x="-13.208" y="-1179.576" size="1.27" layer="25" ratio="10"/>
+<attribute name="SPICEPREFIX" value="C" x="-16.51" y="-1182.37" size="1.778" layer="27" display="off"/>
+<attribute name="VALUE" x="-18.796" y="-1185.418" size="1.27" layer="27" ratio="10"/>
+</element>
+<element name="U$1" library="Parts" library_urn="urn:adsk.eagle:library:2304016" package="POWER_JACK_PTH" package3d_urn="urn:adsk.eagle:package:2338719/2" value="DC-JACK" x="-30.48" y="-1186.18" smashed="yes">
+<attribute name="NAME" x="-31.8516" y="-1184.3512" size="0.6096" layer="25" font="vector" ratio="20"/>
+<attribute name="VALUE" x="-32.2326" y="-1185.3672" size="0.6096" layer="27" font="vector" ratio="20"/>
+</element>
+<element name="C6" library="rcl" library_urn="urn:adsk.eagle:library:334" package="C050-024X044" package3d_urn="urn:adsk.eagle:package:23643/1" value="100n" x="-31.75" y="469.9" smashed="yes">
+<attribute name="MOUSER" value="594-K104K15X7RF53H5" x="-31.75" y="-1191.26" size="1.778" layer="27" display="off"/>
+<attribute name="NAME" x="-33.909" y="471.297" size="1.27" layer="25" ratio="10"/>
+<attribute name="SPICEPREFIX" value="C" x="-31.75" y="-1191.26" size="1.778" layer="27" display="off"/>
+<attribute name="VALUE" x="-33.909" y="467.233" size="1.27" layer="27" ratio="10"/>
+</element>
 </elements>
 <signals>
@@
 <contactref element="LED3" pad="K"/>
 <contactref element="LED2" pad="K"/>
+<contactref element="C6" pad="2"/>
+<contactref element="C1" pad="-"/>
+<contactref element="U$1" pad="GNDBREAK"/>
+<contactref element="U$1" pad="GND"/>
+<wire x1="-25.78" y1="-1175.48" x2="-30.48" y2="-1178.48" width="0" layer="19" extent="1-1"/>
+<wire x1="-14.732" y1="-1182.37" x2="-25.78" y2="-1175.48" width="0" layer="19" extent="1-1"/>
+<wire x1="-16.73" y1="-818" x2="-25.78" y2="-1175.48" width="0" layer="19" extent="1-1"/>
 <wire x1="-16.73" y1="-813" x2="-16.73" y2="-818" width="0" layer="19" extent="1-1"/>
 <wire x1="-16.73" y1="-808" x2="-16.73" y2="-813" width="0" layer="19" extent="1-1"/>
@@
 <wire x1="-19.81" y1="-755" x2="-19.81" y2="-759" width="0" layer="19" extent="1-1"/>
 <wire x1="-19.81" y1="-751" x2="-19.81" y2="-755" width="0" layer="19" extent="1-1"/>
+<wire x1="-29.21" y1="469.9" x2="-30.48" y2="-1178.48" width="0" layer="19" extent="1-1"/>
 </signal>
 <signal name="N$22">
@@
 <wire x1="-12.19" y1="437" x2="-16.73" y2="189" width="0" layer="19" extent="1-1"/>
 </signal>
+<signal name="VCC">
+<contactref element="C1" pad="+"/>
+<contactref element="U$1" pad="PWR"/>
+<contactref element="C6" pad="1"/>
+<wire x1="-18.288" y1="-1182.37" x2="-30.48" y2="-1172.48" width="0" layer="19" extent="1-1"/>
+<wire x1="-34.29" y1="469.9" x2="-30.48" y2="-1172.48" width="0" layer="19" extent="1-1"/>
+</signal>
 </signals>

Commit message: layed out components on board
Parts:
- added ID:C7: 100n, rcl:C050-024X044
- added ID:RN1, ID:RN2: (no value), resistor-sil:SIL9
- added OUT:R10, OUT:R11, OUT:R12, OUT:R13, OUT:R14, OUT:R15, OUT:R8, OUT:R9: 220, rcl:0204/7
- MAR:LED1, MAR:LED2, MAR:LED3, MAR:LED4: value RED -> BLUE
- moved U$1 1490.0 mm to (80.0, 299.7), turned to 180 degrees
- moved C1 1464.5 mm to (73.7, 279.4), turned to 180 degrees
- moved ALU:C6 1356.9 mm to (127.0, 182.2)
- moved ALU:C7 1341.1 mm to (127.0, 159.4)
- moved ALU:IC6 1333.0 mm to (127.0, 193.0), turned to 90 degrees
- moved ALU:C5 1332.8 mm to (92.7, 168.3)
- moved R16 1327.7 mm to (50.5, 261.0), turned to 270 degrees
- moved R15 1323.9 mm to (55.6, 261.0), turned to 270 degrees
- moved ALU:IC7 1321.2 mm to (127.0, 170.2), turned to 90 degrees
- moved R14 1320.2 mm to (60.6, 261.0), turned to 270 degrees
- moved ALU:C4 1318.0 mm to (104.1, 159.4)
- moved R13 1316.5 mm to (65.7, 261.0), turned to 270 degrees
- moved R12 1312.9 mm to (70.8, 261.0), turned to 270 degrees
- moved R11 1309.2 mm to (75.9, 261.0), turned to 270 degrees
- moved R10 1305.6 mm to (81.0, 261.0), turned to 270 degrees
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Connections:
- new net OUT:N$17: OUT:IC1.14, OUT:R12.2
- new net OUT:SEG_AO: OUT:IC1.9, OUT:R8.2
- new net OUT:SEG_BO: OUT:IC1.10, OUT:R9.2
- new net OUT:SEG_CO: OUT:IC1.11, OUT:R10.2
- new net OUT:SEG_DO: OUT:IC1.13, OUT:R11.2
- new net OUT:SEG_DPO: OUT:IC1.17, OUT:R15.2
- new net OUT:SEG_FO: OUT:IC1.15, OUT:R13.2
- new net OUT:SEG_GO: OUT:IC1.16, OUT:R14.2
- net ID:GND: now also ID:C7.2
- net ID:VCC: now also ID:C7.1
- net OUT:SEG_A: now also OUT:R8.1; no longer OUT:IC1.9
- net OUT:SEG_B: now also OUT:R9.1; no longer OUT:IC1.10
- net OUT:SEG_C: now also OUT:R10.1; no longer OUT:IC1.11
- net OUT:SEG_D: now also OUT:R11.1; no longer OUT:IC1.13
- net OUT:SEG_DP: now also OUT:R15.1; no longer OUT:IC1.17
- net OUT:SEG_E: now also OUT:R12.1; no longer OUT:IC1.14
- net OUT:SEG_F: now also OUT:R13.1; no longer OUT:IC1.15
- net OUT:SEG_G: now also OUT:R14.1; no longer OUT:IC1.16
Routing:
- net N$5: track 32.9 -> 0.00 mm
- net N$1: track 52.0 -> 24.3 mm
- net N$2: track 45.5 -> 20.8 mm
- net N$3: track 42.6 -> 18.6 mm
- net N$4: track 38.9 -> 16.4 mm
- net N$8: track 30.4 -> 14.5 mm
- net N$7: track 28.3 -> 18.1 mm
- net !AI: track 29.0 -> 20.1 mm
- net N$22: track 31.8 -> 24.4 mm
- net CLR: track 50.7 -> 44.2 mm
- net N$6: track 25.0 -> 21.7 mm
- net N$15: track 31.6 -> 30.3 mm
- net N$16: track 33.3 -> 32.0 mm
- net N$12: track 23.9 -> 24.6 mm
- net N$11: track 52.3 -> 53.0 mm
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Other:
- board size 100 x 100 mm -> 135 x 300 mm

Commit message: replace most discrete resistors with networks
Parts:
- removed ALU:R1, ALU:R2, ALU:R3, ALU:R4, ALU:R5, ALU:R6, ALU:R7, ALU:R8, ID:R1, ID:R10, ID:R11, ID:R12, ID:R13, ID:R14, ID:R15, ID:R16, ID:R2, ID:R21, ID:R22, ID:R23, ID:R24, ID:R25, ID:R3, ID:R4, ID:R5, ID:R6, ID:R7, ID:R8, ID:R9, IR:R1, IR:R2, IR:R3, IR:R4, IR:R5, IR:R6, IR:R7, IR:R8, MAR:R1, MAR:R2, MAR:R3, MAR:R4, OUT:R10, OUT:R11, OUT:R12, OUT:R13, OUT:R14, OUT:R15, OUT:R8, OUT:R9, PC:R1, PC:R2, PC:R3, PC:R4, R10, R11, R12, R13, R14, R15, R16, R9, RA:R1, RA:R2, RA:R3, RA:R4, RA:R5, RA:R6, RA:R7, RA:R8, RAM:R1, RAM:R2, RAM:R3, RAM:R4, RAM:R5, RAM:R6, RAM:R7, RAM:R8, RB:R1, RB:R2, RB:R3, RB:R4, RB:R5, RB:R6, RB:R7, RB:R8: 220, rcl:0204/7
- removed R1, R2, R3, R4, R5, R6, R7, R8: 10k, rcl:0204/7
- added ALU:RN3, ID:RN3, IR:RN3, RA:RN3, RAM:RN3, RB:RN3, RN3: 220, resistor-sil:SIL9
- added MAR:RN1, PC:RN1: 220, resistor-sil:SIL5
- added OUT:RN1, OUT:RN2: 220, resistor-sil:SIL8
- added RN1: 10k, resistor-sil:SIL9
- C1: value (none) -> 100u
- ID:RN1, ID:RN2: value (none) -> 220
- OUT:D1, OUT:D2, OUT:D3, OUT:D4: value (none) -> RED
- moved ID:RN1 83.8 mm to (92.4, 22.2)
- moved ID:RN2 81.8 mm to (92.4, 9.53)
- moved ID:S1 2.54 mm to (30.5, 33.0)
Connections:
- net OUT:N$16 renamed OUT:N$10
- removed net ID:N$32: ID:FI.A
- removed net IR:D5: IR:IC3.14
- removed net IR:D6: IR:IC3.13
- removed net IR:D7: IR:IC3.12
- removed net IR:D8: IR:IC3.11
- removed net IR:N$4: IR:R1.1, IR:R2.1, IR:R3.1, IR:R4.1, IR:R5.1, IR:R6.1, IR:R7.1, IR:R8.1
- net ALU:GND: now also ALU:RN3.1; no longer ALU:R1.1, ALU:R2.1, ALU:R3.1, ALU:R4.1, ALU:R5.1, ALU:R6.1, ALU:R7.1, ALU:R8.1
- net ALU:N$10: now also ALU:RN3.7; no longer ALU:R6.2
- net ALU:N$11: now also ALU:RN3.6; no longer ALU:R5.2
- net ALU:N$12: now also ALU:RN3.5; no longer ALU:R4.2
- net ALU:N$13: now also ALU:RN3.4; no longer ALU:R3.2
- net ALU:N$14: now also ALU:RN3.3; no longer ALU:R2.2
- net ALU:N$15: now also ALU:RN3.2; no longer ALU:R1.2
- net ALU:N$8: now also ALU:RN3.9; no longer ALU:R8.2
- net ALU:N$9: now also ALU:RN3.8; no longer ALU:R7.2
- net D1: now also LED1.A, RN1.9; no longer R1.2, R9.2
- net D2: now also LED2.A, RN1.8; no longer R10.2, R2.2
- net D3: now also LED3.A, RN1.7; no longer R11.2, R3.2
- net D4: now also LED4.A, RN1.6; no longer R12.2, R4.2
- net D5: now also IR:IC3.14, LED5.A, RN1.5; no longer R13.2, R5.2
- net D6: now also IR:IC3.13, LED6.A, RN1.4; no longer R14.2, R6.2
- net D7: now also IR:IC3.12, LED7.A, RN1.3; no longer R15.2, R7.2
- net D8: now also IR:IC3.11, LED8.A, RN1.2; no longer R16.2, R8.2
- net GND: now also RN1.1, RN3.1; no longer LED1.K, LED2.K, LED3.K, LED4.K, LED5.K, LED6.K, LED7.K, LED8.K, R1.1, R2.1, R3.1, R4.1, R5.1, R6.1, R7.1, R8.1
- net ID:GND: now also ID:IC5.3, ID:IC5.4, ID:IC5.5, ID:IC5.6, ID:RN1.1, ID:RN2.1, ID:RN3.1; no longer ID:R1.1, ID:R10.1, ID:R11.1, ID:R12.1, ID:R13.1, ID:R14.1, ID:R15.1, ID:R16.1, ID:R2.1, ID:R21.1, ID:R22.1, ID:R23.1, ID:R24.1, ID:R25.1, ID:R3.1, ID:R4.1, ID:R5.1, ID:R6.1, ID:R7.1, ID:R8.1, ID:R9.1
- net ID:N$1: now also ID:RN1.2; no longer ID:R1.2
- net ID:N$10: now also ID:RN2.3; no longer ID:R10.2
- net ID:N$11: now also ID:RN2.4; no longer ID:R11.2
- net ID:N$12: now also ID:RN2.5; no longer ID:R12.2
- net ID:N$13: now also ID:RN2.6; no longer ID:R13.2
- net ID:N$14: now also ID:RN2.7; no longer ID:R14.2
- net ID:N$15: now also ID:RN2.8; no longer ID:R15.2
- net ID:N$2: now also ID:RN1.3; no longer ID:R2.2
- net ID:N$3: now also ID:RN1.4; no longer ID:R3.2
- net ID:N$30: now also ID:FI.A
- net ID:N$31: now also ID:RN2.9; no longer ID:R16.2
- net ID:N$33: now also ID:RN3.4; no longer ID:R23.2
- net ID:N$34: now also ID:RN3.2; no longer ID:R25.2
- net ID:N$35: now also ID:RN3.3; no longer ID:R24.2
- net ID:N$36: now also ID:RN3.5; no longer ID:R22.2
- net ID:N$37: now also ID:RN3.6; no longer ID:R21.2
- net ID:N$4: now also ID:RN1.5; no longer ID:R4.2
- net ID:N$5: now also ID:RN1.6; no longer ID:R5.2
- net ID:N$6: now also ID:RN1.7; no longer ID:R6.2
- net ID:N$7: now also ID:RN1.8; no longer ID:R7.2
- net ID:N$8: now also ID:RN1.9; no longer ID:R8.2
- net ID:N$9: now also ID:RN2.2; no longer ID:R9.2
- net IR:GND: now also IR:RN3.1
- net IR:N$1: now also IR:RN3.9; no longer IR:R8.2
- net IR:N$2: now also IR:RN3.8; no longer IR:R7.2
- net IR:N$3: now also IR:RN3.7; no longer IR:R6.2
- net IR:N$5: now also IR:RN3.6; no longer IR:R5.2
- net IR:N$6: now also IR:RN3.5; no longer IR:R4.2
- net IR:N$7: now also IR:RN3.4; no longer IR:R3.2
- net IR:N$8: now also IR:RN3.3; no longer IR:R2.2
- net IR:N$9: now also IR:RN3.2; no longer IR:R1.2
- net MAR:GND: now also MAR:RN1.1; no longer MAR:R1.1, MAR:R2.1, MAR:R3.1, MAR:R4.1
- net MAR:N$10: now also MAR:RN1.2; no longer MAR:R1.2
- net MAR:N$2: now also MAR:RN1.5; no longer MAR:R4.2
- net MAR:N$4: now also MAR:RN1.4; no longer MAR:R3.2
- net MAR:N$8: now also MAR:RN1.3; no longer MAR:R2.2
- net N$23: now also LED8.K, RN3.2; no longer LED1.A, R9.1
- net N$24: now also LED7.K, RN3.3; no longer LED2.A, R10.1
- net N$25: now also LED6.K, RN3.4; no longer LED3.A, R11.1
- net N$26: now also LED5.K, RN3.5; no longer LED4.A, R12.1
- net N$27: now also LED4.K, RN3.6; no longer LED5.A, R13.1
- net N$28: now also LED3.K, RN3.7; no longer LED6.A, R14.1
- net N$29: now also LED2.K, RN3.8; no longer LED7.A, R15.1
- net N$30: now also LED1.K, RN3.9; no longer LED8.A, R16.1
- net OUT:N$17: now also OUT:RN2.1; no longer OUT:R12.2
- net OUT:SEG_A: now also OUT:RN1.6; no longer OUT:R8.1
- net OUT:SEG_AO: now also OUT:RN1.5; no longer OUT:R8.2
- net OUT:SEG_B: now also OUT:RN1.8; no longer OUT:R9.1
- net OUT:SEG_BO: now also OUT:RN1.7; no longer OUT:R9.2
- net OUT:SEG_C: now also OUT:RN2.6; no longer OUT:R10.1
- net OUT:SEG_CO: now also OUT:RN2.5; no longer OUT:R10.2
- net OUT:SEG_D: now also OUT:RN2.4; no longer OUT:R11.1
- net OUT:SEG_DO: now also OUT:RN2.3; no longer OUT:R11.2
- net OUT:SEG_DP: now also OUT:RN2.8; no longer OUT:R15.1
- net OUT:SEG_DPO: now also OUT:RN2.7; no longer OUT:R15.2
- net OUT:SEG_E: now also OUT:RN2.2; no longer OUT:R12.1
- net OUT:SEG_F: now also OUT:RN1.4; no longer OUT:R13.1
- net OUT:SEG_FO: now also OUT:RN1.3; no longer OUT:R13.2
- net OUT:SEG_G: now also OUT:RN1.2; no longer OUT:R14.1
- net OUT:SEG_GO: now also OUT:RN1.1; no longer OUT:R14.2
- net PC:GND: now also PC:RN1.1; no longer PC:R1.1, PC:R2.1, PC:R3.1, PC:R4.1
- net PC:N$1: now also PC:RN1.5; no longer PC:R4.2
- net PC:N$2: now also PC:RN1.4; no longer PC:R3.2
- net PC:N$3: now also PC:RN1.3; no longer PC:R2.2
- net PC:N$4: now also PC:RN1.2; no longer PC:R1.2
- net RA:GND: now also RA:RN3.1; no longer RA:R1.1, RA:R2.1, RA:R3.1, RA:R4.1, RA:R5.1, RA:R6.1, RA:R7.1, RA:R8.1
- net RA:N$1: now also RA:RN3.2; no longer RA:R1.2
- net RA:N$2: now also RA:RN3.3; no longer RA:R2.2
- net RA:N$3: now also RA:RN3.4; no longer RA:R3.2
- net RA:N$4: now also RA:RN3.5; no longer RA:R4.2
- net RA:N$5: now also RA:RN3.6; no longer RA:R5.2
- net RA:N$6: now also RA:RN3.7; no longer RA:R6.2
- net RA:N$7: now also RA:RN3.8; no longer RA:R7.2
- net RA:N$8: now also RA:RN3.9; no longer RA:R8.2
- net RAM:GND: now also RAM:IC8.10, RAM:IC8.11, RAM:IC8.13, RAM:IC8.14, RAM:IC8.5, RAM:IC8.6, RAM:RN3.1; no longer RAM:R1.1, RAM:R2.1, RAM:R3.1, RAM:R4.1, RAM:R5.1, RAM:R6.1, RAM:R7.1, RAM:R8.1
- net RAM:N$10: now also RAM:RN3.8; no longer RAM:R7.2
- net RAM:N$11: now also RAM:RN3.7; no longer RAM:R6.2
- net RAM:N$12: now also RAM:RN3.6; no longer RAM:R5.2
- net RAM:N$13: now also RAM:RN3.5; no longer RAM:R4.2
- net RAM:N$14: now also RAM:RN3.4; no longer RAM:R3.2
- net RAM:N$15: now also RAM:RN3.3; no longer RAM:R2.2
- net RAM:N$16: now also RAM:RN3.2; no longer RAM:R1.2
- net RAM:N$9: now also RAM:RN3.9; no longer RAM:R8.2
- net RB:GND: now also RB:RN3.1; no longer RB:R1.1, RB:R2.1, RB:R3.1, RB:R4.1, RB:R5.1, RB:R6.1, RB:R7.1, RB:R8.1
- net RB:N$1: now also RB:RN3.9; no longer RB:R8.2
- net RB:N$2: now also RB:RN3.8; no longer RB:R7.2
- net RB:N$3: now also RB:RN3.7; no longer RB:R6.2
- net RB:N$4: now also RB:RN3.6; no longer RB:R5.2
- net RB:N$5: now also RB:RN3.5; no longer RB:R4.2
- net RB:N$6: now also RB:RN3.4; no longer RB:R3.2
- net RB:N$7: now also RB:RN3.3; no longer RB:R2.2
- net RB:N$8: now also RB:RN3.2; no longer RB:R1.2
- net SR:GND: now also SR:IC2.11, SR:IC2.12

Commit message: started routing of modules
Parts:
- removed CLK:R2: 1M, rcl:RTRIM64W
- added CLK:RV2: (no value), SparkFun-Electromechanical:ALPS_POT_KIT
- added MAR:R1: 10k, rcl:0204/7
- added MAR:RN2: 10k, resistor-sil:SIL5
- added RAM:RN1: 10k, resistor-sil:SIL9
- moved RAM:S1 95.4 mm to (21.6, 111.8), turned to 270 degrees
- moved RAM:S2 79.1 mm to (14.0, 192.1)
- moved MAR:C1 42.1 mm to (5.71, 233.7)
- moved MAR:IC1 42.1 mm to (17.8, 233.7)
- moved RA:LED8 32.6 mm to (88.9, 255.3)
- moved MAR:PROG 32.4 mm to (11.4, 203.2)
- moved MAR:R10 32.4 mm to (15.9, 210.2)
- moved MAR:R9 32.4 mm to (11.4, 210.2)
- moved MAR:RUN 32.4 mm to (15.9, 203.2)
- moved ALU:C3 32.3 mm to (127.0, 159.4)
- moved MAR:S3 31.8 mm to (6.35, 207.0)
- moved OUT:RN1 31.8 mm to (114.3, 106.7)
- moved RA:LED1 30.1 mm to (120.0, 255.3)
- moved RAM:C1 27.9 mm to (21.6, 121.3)
- moved RAM:C6 27.9 mm to (8.89, 121.3)
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Connections:
- net N$22 renamed CLK
- net N$36 renamed !CLK
- removed net MAR:N$6: MAR:IC2.14, MAR:S1.5
- new net MAR:N$11: MAR:IC2.14, MAR:RN2.5, MAR:S1.5
- net CLK:N$1: now also CLK:RV2.P$2, CLK:RV2.P$3; no longer CLK:R2.1, CLK:R2.2
- net CLK:N$3: now also CLK:RV2.P$1; no longer CLK:R2.3
- net MAR:N$1: now also MAR:RN2.2
- net MAR:N$3: now also MAR:RN2.3
- net MAR:N$5: now also MAR:RN2.4
- net MAR:VCC: now also MAR:R1.1, MAR:RN2.1
- net N$21: now also MAR:R1.2
- net RAM:N$18: now also RAM:RN1.9
- net RAM:N$19: now also RAM:RN1.8
- net RAM:N$20: now also RAM:RN1.7
- net RAM:N$21: now also RAM:RN1.6
- net RAM:N$22: now also RAM:RN1.5
- net RAM:N$23: now also RAM:RN1.4
- net RAM:N$24: now also RAM:RN1.3
- net RAM:N$25: now also RAM:RN1.2
- net RAM:VCC: now also RAM:RN1.1
Routing:
- net D4: track 0.00 -> 183.3 mm, vias 0 -> 2
- net D3: track 0.00 -> 171.1 mm, vias 0 -> 2
- net D2: track 0.00 -> 159.9 mm, vias 0 -> 2
- net D1: track 0.00 -> 151.8 mm, vias 0 -> 2
- net N$5: track 0.00 -> 145.1 mm
- net N$7: track 18.1 -> 143.6 mm
- net N$8: track 14.5 -> 137.1 mm
- net N$6: track 21.7 -> 135.6 mm
- net D8: track 0.00 -> 109.4 mm, vias 0 -> 2
- net D7: track 0.00 -> 107.0 mm, vias 0 -> 2
- net N$2: track 20.8 -> 117.0 mm
- net D5: track 0.00 -> 91.4 mm, vias 0 -> 2
- net N$21: track 0.00 -> 89.6 mm, vias 0 -> 1
- net D6: track 0.00 -> 87.6 mm
- net N$3: track 18.6 -> 105.6 mm
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
Commit message: routed seperate modules except power nets
Parts:
- SR:LED1, SR:LED2: value RED -> BLUE
- moved RAM:IC8 86.9 mm to (24.1, 198.1), turned to 90 degrees
- moved RAM:R9 84.7 mm to (14.0, 199.1)
- moved RAM:C10 83.8 mm to (15.2, 202.2), turned to 180 degrees
- moved OUT:RN1 78.4 mm to (120.7, 28.6)
- moved RAM:C8 73.2 mm to (24.1, 186.1), turned to 0 degrees
- moved RAM:S1 70.0 mm to (48.3, 176.5)
- moved OUT:RN2 56.8 mm to (100.3, 28.6)
- moved MAR:C1 56.2 mm to (35.6, 186.1), turned to 0 degrees
- moved MAR:C2 54.1 mm to (47.0, 186.1), turned to 0 degrees
- moved OUT:D2 53.7 mm to (111.8, 41.9)
- moved OUT:D3 53.7 mm to (99.1, 41.9)
- moved OUT:D1 53.7 mm to (124.5, 41.9)
- moved OUT:D4 53.7 mm to (86.4, 41.9)
- moved SR:LED1 53.4 mm to (5.71, 94.0)
- moved SR:LED2 53.4 mm to (10.2, 94.0)
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Routing:
- net D1: track 151.8 -> 365.7 mm, vias 2 -> 7
- net D2: track 159.9 -> 361.3 mm, vias 2 -> 7
- net D3: track 171.1 -> 359.5 mm, vias 2 -> 9
- net D5: track 91.4 -> 279.7 mm, vias 2 -> 6
- net D4: track 183.3 -> 369.8 mm, vias 2 -> 9
- net D6: track 87.6 -> 270.7 mm, vias 0 -> 4
- net D7: track 107.0 -> 287.6 mm, vias 2 -> 7
- net D8: track 109.4 -> 289.3 mm, vias 2 -> 6
- net ZF: track 0.00 -> 123.2 mm, vias 0 -> 4
- net CF: track 0.00 -> 116.3 mm, vias 0 -> 4
- net ID:N$26: track 0.00 -> 96.3 mm, vias 0 -> 3
- net ID:MI2: track 0.00 -> 91.4 mm, vias 0 -> 4
- net OUT:DIG4: track 0.00 -> 91.3 mm, vias 0 -> 1
- net ID:N$28: track 0.00 -> 90.0 mm, vias 0 -> 4
- net N$2: track 117.0 -> 27.1 mm, vias 0 -> 1
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