File: Board/SAP-1.brd (EAGLE design)
At the start: 135 x 300 mm, 233 parts

Commit message: added first routing pass
Parts:
- moved RAM:R9 94.9 mm to (35.6, 106.7), turned to 180 degrees
- moved RAM:C10 94.8 mm to (35.2, 109.5)
- moved OUT:C7 2.03 mm to (94.0, 55.6)
- moved OUT:C8 1.27 mm to (85.1, 69.2)
- moved OUT:C4 1.27 mm to (85.1, 55.2)
- moved OUT:IC4 1.27 mm to (85.1, 62.2)
- moved OUT:RN1 0.63 mm to (120.7, 27.9)
- moved OUT:RN2 0.63 mm to (100.3, 27.9)
- turned PC:C2 to 180 degrees
- turned RB:C2 to 0 degrees
- turned RB:C3 to 0 degrees
Connections:
- removed net ALU:GND: ALU:C1.2, ALU:C2.2, ALU:C3.2, ALU:C4.2, ALU:C5.2, ALU:C6.2, ALU:C7.2, ALU:IC1.8, ALU:IC2.8, ALU:IC3.7, ALU:IC4.7, ALU:IC5.10, ALU:IC6.7, ALU:IC7.7, ALU:RN3.1
- removed net ALU:VCC: ALU:C1.1, ALU:C2.1, ALU:C3.1, ALU:C4.1, ALU:C5.1, ALU:C6.1, ALU:C7.1, ALU:IC1.16, ALU:IC2.16, ALU:IC3.14, ALU:IC4.14, ALU:IC5.1, ALU:IC5.20, ALU:IC6.14, ALU:IC7.14
- removed net CLK:GND: CLK:C1.-, CLK:C2.2, CLK:C3.2, CLK:C4.2, CLK:C5.2, CLK:C6.2, CLK:C7.2, CLK:C8.2, CLK:IC2.1, CLK:IC3.1, CLK:IC4.1, CLK:IC4.6, CLK:IC5.7, CLK:IC6.7, CLK:IC7.7, CLK:R11.1, CLK:S1.1, CLK:S2.2
- removed net CLK:VCC: CLK:C3.1, CLK:C6.1, CLK:C8.1, CLK:IC2.4, CLK:IC2.8, CLK:IC3.4, CLK:IC3.8, CLK:IC4.8, CLK:IC5.14, CLK:IC6.14, CLK:IC7.14, CLK:R1.2, CLK:R10.2, CLK:R5.2, CLK:R6.2, CLK:R9.2
- removed net ID:GND: ID:C1.2, ID:C2.2, ID:C3.2, ID:C4.2, ID:C5.2, ID:C6.2, ID:C7.2, ID:IC1.1, ID:IC1.12, ID:IC1.18, ID:IC1.19, ID:IC1.20, ID:IC2.12, ID:IC2.18, ID:IC2.19, ID:IC2.20, ID:IC3.7, ID:IC4.7, ID:IC5.3, ID:IC5.4, ID:IC5.5, ID:IC5.6, ID:IC5.8, ID:IC6.4, ID:IC6.5, ID:IC6.8, ID:IC7.7, ID:R17.1, ID:RN1.1, ID:RN2.1, ID:RN3.1
- removed net ID:VCC: ID:C1.1, ID:C2.1, ID:C3.1, ID:C4.1, ID:C5.1, ID:C6.1, ID:C7.1, ID:IC1.21, ID:IC1.24, ID:IC2.1, ID:IC2.21, ID:IC2.24, ID:IC3.14, ID:IC4.14, ID:IC5.10, ID:IC5.16, ID:IC5.7, ID:IC5.9, ID:IC6.16, ID:IC6.6, ID:IC7.14, ID:S1.1
- removed net IR:GND: IR:C1.2, IR:C2.2, IR:C3.2, IR:IC1.10, IR:IC2.1, IR:IC2.2, IR:IC2.8, IR:IC3.1, IR:IC3.2, IR:IC3.8, IR:RN3.1
- removed net IR:VCC: IR:C1.1, IR:C2.1, IR:C3.1, IR:IC1.1, IR:IC1.20, IR:IC2.16, IR:IC3.16
- removed net MAR:GND: MAR:C1.2, MAR:C2.2, MAR:IC1.1, MAR:IC1.2, MAR:IC1.8, MAR:IC2.15, MAR:IC2.8, MAR:RN1.1, MAR:S1.1, MAR:S1.2, MAR:S1.3, MAR:S1.4, MAR:S3.2
- removed net MAR:VCC: MAR:C1.1, MAR:C2.1, MAR:IC1.16, MAR:IC2.16, MAR:PROG.A, MAR:R1.1, MAR:RN2.1, MAR:RUN.A
- removed net OUT:GND: OUT:C1.2, OUT:C2.2, OUT:C3.2, OUT:C4.2, OUT:C5.2, OUT:C6.2, OUT:C7.2, OUT:C8.2, OUT:IC1.12, OUT:IC1.18, OUT:IC1.20, OUT:IC2.7, OUT:IC3.10, OUT:IC4.1, OUT:IC5.13, OUT:IC6.1, OUT:IC6.8, OUT:S3.1
- removed net OUT:VCC: OUT:C1.1, OUT:C2.1, OUT:C3.1, OUT:C4.1, OUT:C5.1, OUT:C6.1, OUT:IC1.21, OUT:IC1.24, OUT:IC2.14, OUT:IC3.20, OUT:IC4.4, OUT:IC4.8, OUT:IC5.12, OUT:IC5.16, OUT:IC5.2, OUT:IC5.3, OUT:IC5.4, OUT:IC5.5, OUT:IC5.7, OUT:IC5.8, OUT:IC5.9, OUT:IC6.16, OUT:R1.2, OUT:S3.3
- removed net PC:GND: PC:C1.2, PC:C2.2, PC:IC1.8, PC:IC2.10, PC:IC2.6, PC:IC2.7, PC:IC2.8, PC:IC2.9, PC:RN1.1
- removed net PC:VCC: PC:C1.1, PC:C2.1, PC:IC1.16, PC:IC2.1, PC:IC2.20
- removed net RA:GND: RA:C1.2, RA:C2.2, RA:C3.2, RA:IC1.10, RA:IC2.1, RA:IC2.2, RA:IC2.8, RA:IC3.1, RA:IC3.2, RA:IC3.8, RA:RN3.1
- removed net RA:VCC: RA:C1.1, RA:C2.1, RA:C3.1, RA:IC1.1, RA:IC1.20, RA:IC2.16, RA:IC3.16
- removed net RAM:GND: RAM:C1.2, RAM:C2.2, RAM:C3.2, RAM:C4.2, RAM:C5.2, RAM:C6.2, RAM:C7.2, RAM:C8.2, RAM:C9.2, RAM:IC1.2, RAM:IC1.8, RAM:IC2.2, RAM:IC2.8, RAM:IC3.10, RAM:IC4.7, RAM:IC5.7, RAM:IC6.15, RAM:IC6.8, RAM:IC7.15, RAM:IC7.8, RAM:IC8.10, RAM:IC8.11, RAM:IC8.13, RAM:IC8.14, RAM:IC8.15, RAM:IC8.5, RAM:IC8.6, RAM:IC8.8, RAM:IC9.7, RAM:R9.1, RAM:RN3.1, RAM:S1.1, RAM:S2.1, RAM:S2.2, RAM:S2.3, RAM:S2.4, RAM:S2.5, RAM:S2.6, RAM:S2.7, RAM:S2.8
- removed net RAM:VCC: RAM:C1.1, RAM:C2.1, RAM:C3.1, RAM:C4.1, RAM:C5.1, RAM:C6.1, RAM:C7.1, RAM:C8.1, RAM:C9.1, RAM:IC1.16, RAM:IC2.16, RAM:IC3.1, RAM:IC3.20, RAM:IC4.14, RAM:IC5.14, RAM:IC6.16, RAM:IC7.16, RAM:IC8.16, RAM:IC9.14, RAM:RN1.1
- removed net RB:GND: RB:C1.2, RB:C2.2, RB:C3.2, RB:IC1.10, RB:IC2.1, RB:IC2.2, RB:IC2.8, RB:IC3.1, RB:IC3.2, RB:IC3.8, RB:RN3.1
- removed net RB:VCC: RB:C1.1, RB:C2.1, RB:C3.1, RB:IC1.1, RB:IC1.20, RB:IC2.16, RB:IC3.16
- removed net SR:GND: SR:C1.2, SR:IC2.1, SR:IC2.11, SR:IC2.12, SR:IC2.2, SR:IC2.8, SR:R1.1, SR:R2.1
- removed net SR:VCC: SR:C1.1, SR:IC2.16
- net GND: now also ALU:C1.2, ALU:C2.2, ALU:C3.2, ALU:C4.2, ALU:C5.2, ALU:C6.2, ALU:C7.2, ALU:IC1.8, ALU:IC2.8, ALU:IC3.7, ALU:IC4.7, ALU:IC5.10, ALU:IC6.7, ALU:IC7.7, ALU:RN3.1, CLK:C1.-, CLK:C2.2, CLK:C3.2, CLK:C4.2, CLK:C5.2, CLK:C6.2, CLK:C7.2, CLK:C8.2, CLK:IC2.1, CLK:IC3.1, CLK:IC4.1, CLK:IC4.6, CLK:IC5.7, CLK:IC6.7, CLK:IC7.7, CLK:R11.1, CLK:S1.1, CLK:S2.2, ID:C1.2, ID:C2.2, ID:C3.2, ID:C4.2, ID:C5.2, ID:C6.2, ID:C7.2, ID:IC1.1, ID:IC1.12, ID:IC1.18, ID:IC1.19, ID:IC1.20, ID:IC2.12, ID:IC2.18, ID:IC2.19, ID:IC2.20, ID:IC3.7, ID:IC4.7, ID:IC5.3, ID:IC5.4, ID:IC5.5, ID:IC5.6, ID:IC5.8, ID:IC6.4, ID:IC6.5, ID:IC6.8, ID:IC7.7, ID:R17.1, ID:RN1.1, ID:RN2.1, ID:RN3.1, IR:C1.2, IR:C2.2, IR:C3.2, IR:IC1.10, IR:IC2.1, IR:IC2.2, IR:IC2.8, IR:IC3.1, IR:IC3.2, IR:IC3.8, IR:RN3.1, MAR:C1.2, MAR:C2.2, MAR:IC1.1, MAR:IC1.2, MAR:IC1.8, MAR:IC2.15, MAR:IC2.8, MAR:RN1.1, MAR:S1.1, MAR:S1.2, MAR:S1.3, MAR:S1.4, MAR:S3.2, OUT:C1.2, OUT:C2.2, OUT:C3.2, OUT:C4.2, OUT:C5.2, OUT:C6.2, OUT:C7.2, OUT:C8.2, OUT:IC1.12, OUT:IC1.18, OUT:IC1.20, OUT:IC2.7, OUT:IC3.10, OUT:IC4.1, OUT:IC5.13, OUT:IC6.1, OUT:IC6.8, OUT:S3.1, PC:C1.2, PC:C2.2, PC:IC1.8, PC:IC2.10, PC:IC2.6, PC:IC2.7, PC:IC2.8, PC:IC2.9, PC:RN1.1, RA:C1.2, RA:C2.2, RA:C3.2, RA:IC1.10, RA:IC2.1, RA:IC2.2, RA:IC2.8, RA:IC3.1, RA:IC3.2, RA:IC3.8, RA:RN3.1, RAM:C1.2, RAM:C2.2, RAM:C3.2, RAM:C4.2, RAM:C5.2, RAM:C6.2, RAM:C7.2, RAM:C8.2, RAM:C9.2, RAM:IC1.2, RAM:IC1.8, RAM:IC2.2, RAM:IC2.8, RAM:IC3.10, RAM:IC4.7, RAM:IC5.7, RAM:IC6.15, RAM:IC6.8, RAM:IC7.15, RAM:IC7.8, RAM:IC8.10, RAM:IC8.11, RAM:IC8.13, RAM:IC8.14, RAM:IC8.15, RAM:IC8.5, RAM:IC8.6, RAM:IC8.8, RAM:IC9.7, RAM:R9.1, RAM:RN3.1, RAM:S1.1, RAM:S2.1, RAM:S2.2, RAM:S2.3, RAM:S2.4, RAM:S2.5, RAM:S2.6, RAM:S2.7, RAM:S2.8, RB:C1.2, RB:C2.2, RB:C3.2, RB:IC1.10, RB:IC2.1, RB:IC2.2, RB:IC2.8, RB:IC3.1, RB:IC3.2, RB:IC3.8, RB:RN3.1, SR:C1.2, SR:IC2.1, SR:IC2.11, SR:IC2.12, SR:IC2.2, SR:IC2.8, SR:R1.1, SR:R2.1
- net VCC: now also ALU:C1.1, ALU:C2.1, ALU:C3.1, ALU:C4.1, ALU:C5.1, ALU:C6.1, ALU:C7.1, ALU:IC1.16, ALU:IC2.16, ALU:IC3.14, ALU:IC4.14, ALU:IC5.1, ALU:IC5.20, ALU:IC6.14, ALU:IC7.14, CLK:C3.1, CLK:C6.1, CLK:C8.1, CLK:IC2.4, CLK:IC2.8, CLK:IC3.4, CLK:IC3.8, CLK:IC4.8, CLK:IC5.14, CLK:IC6.14, CLK:IC7.14, CLK:R1.2, CLK:R10.2, CLK:R5.2, CLK:R6.2, CLK:R9.2, ID:C1.1, ID:C2.1, ID:C3.1, ID:C4.1, ID:C5.1, ID:C6.1, ID:C7.1, ID:IC1.21, ID:IC1.24, ID:IC2.1, ID:IC2.21, ID:IC2.24, ID:IC3.14, ID:IC4.14, ID:IC5.10, ID:IC5.16, ID:IC5.7, ID:IC5.9, ID:IC6.16, ID:IC6.6, ID:IC7.14, ID:S1.1, IR:C1.1, IR:C2.1, IR:C3.1, IR:IC1.1, IR:IC1.20, IR:IC2.16, IR:IC3.16, MAR:C1.1, MAR:C2.1, MAR:IC1.16, MAR:IC2.16, MAR:PROG.A, MAR:R1.1, MAR:RN2.1, MAR:RUN.A, OUT:C1.1, OUT:C2.1, OUT:C3.1, OUT:C4.1, OUT:C5.1, OUT:C6.1, OUT:IC1.21, OUT:IC1.24, OUT:IC2.14, OUT:IC3.20, OUT:IC4.4, OUT:IC4.8, OUT:IC5.12, OUT:IC5.16, OUT:IC5.2, OUT:IC5.3, OUT:IC5.4, OUT:IC5.5, OUT:IC5.7, OUT:IC5.8, OUT:IC5.9, OUT:IC6.16, OUT:R1.2, OUT:S3.3, PC:C1.1, PC:C2.1, PC:IC1.16, PC:IC2.1, PC:IC2.20, RA:C1.1, RA:C2.1, RA:C3.1, RA:IC1.1, RA:IC1.20, RA:IC2.16, RA:IC3.16, RAM:C1.1, RAM:C2.1, RAM:C3.1, RAM:C4.1, RAM:C5.1, RAM:C6.1, RAM:C7.1, RAM:C8.1, RAM:C9.1, RAM:IC1.16, RAM:IC2.16, RAM:IC3.1, RAM:IC3.20, RAM:IC4.14, RAM:IC5.14, RAM:IC6.16, RAM:IC7.16, RAM:IC8.16, RAM:IC9.14, RAM:RN1.1, RB:C1.1, RB:C2.1, RB:C3.1, RB:IC1.1, RB:IC1.20, RB:IC2.16, RB:IC3.16, SR:C1.1, SR:IC2.16
Routing:
- net VCC: track 0.00 -> 881.4 mm, vias 0 -> 24
- net CLK: track 35.7 -> 562.1 mm, vias 0 -> 12
- net CLR: track 0.00 -> 464.2 mm, vias 0 -> 15
- net !CLR: track 0.00 -> 370.5 mm, vias 0 -> 3
- net !CLK: track 0.00 -> 348.9 mm, vias 0 -> 2
- net !JP: track 0.00 -> 340.3 mm, vias 0 -> 5
- net !CO: track 0.00 -> 317.5 mm, vias 0 -> 4
- net !AI: track 0.00 -> 309.6 mm, vias 0 -> 5
- net ZR: track 0.00 -> 299.9 mm, vias 0 -> 4
- net CE: track 30.2 -> 330.1 mm, vias 1 -> 3
- net HLT: track 20.8 -> 319.8 mm, vias 2 -> 6
- net !MI: track 0.00 -> 287.1 mm, vias 0 -> 4
- net CY: track 0.00 -> 273.1 mm, vias 0 -> 4
- net !AO: track 0.00 -> 250.0 mm, vias 0 -> 3
- net !EO: track 0.00 -> 234.8 mm, vias 0 -> 3
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- added copper zone on layer 16, net GND
- added copper zone on layer 1, net VCC

Commit message: added mounting holes
Parts:
- added H1, H2, H3, H4, H5, H6: MOUNT-PAD-ROUND3.2, holes:3,2-PAD
- moved U$1 16.1 mm to (135.0, 285.7), turned to 90 degrees
- moved OUT:C1 7.62 mm to (130.2, 72.4)
- moved OUT:C3 7.62 mm to (91.1, 78.1)
- moved OUT:C4 7.62 mm to (85.1, 62.9)
- moved OUT:C5 7.62 mm to (125.7, 83.2)
- moved OUT:C6 7.62 mm to (114.3, 83.2)
- moved OUT:D1 7.62 mm to (124.5, 49.5)
- moved OUT:D2 7.62 mm to (111.8, 49.5)
- moved OUT:D3 7.62 mm to (99.1, 49.5)
- moved OUT:D4 7.62 mm to (86.4, 49.5)
- moved OUT:IC1 7.62 mm to (113.0, 72.4)
- moved OUT:IC5 7.62 mm to (125.7, 95.2)
- moved OUT:IC6 7.62 mm to (114.3, 95.2)
- moved ID:AI 7.62 mm to (106.7, 26.0)
- moved ID:AO 7.62 mm to (102.2, 26.0)
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Connections:
- net GND: now also H1.B3,2, H2.B3,2, H3.B3,2, H4.B3,2, H5.B3,2, H6.B3,2
Routing:
- net ZR: track 299.9 -> 282.1 mm
- net CY: track 273.1 -> 255.3 mm
- net !BI: track 224.8 -> 214.7 mm
- net HLT: track 319.8 -> 309.6 mm
- net CLR: track 464.2 -> 454.1 mm
- net !RO: track 192.8 -> 182.7 mm
- net !JP: track 340.3 -> 330.2 mm
- net !EO: track 234.8 -> 224.6 mm
- net !CLR: track 370.5 -> 360.4 mm
- net !AO: track 250.0 -> 239.8 mm
- net RI: track 134.5 -> 124.4 mm
- net SU: track 285.9 -> 275.8 mm
- net CE: track 330.1 -> 319.9 mm
- net !MI: track 287.1 -> 276.9 mm
- net !CO: track 317.5 -> 307.3 mm
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