File: Board/SAP-1.sch (EAGLE design)
At the start: 0 parts

Commit message: added output module
Other:
- note added: "Display D1 -> LSB D4 -> MSB/Sign"
- note added: "Display Decoder"
- note added: "Display Multiplexer"
- note added: "Output Register"

Commit message: connected seperate modules
Parts:
- added LED1, LED2, LED3, LED4, LED5, LED6, LED7, LED8: (no value), led:LED3MM
- added R1, R2, R3, R4, R5, R6, R7, R8: 10k, rcl:R-US_0204/7
Connections:
- new net A1: LED1.A
- new net A2: LED2.A
- new net A3: LED3.A
- new net A4: LED4.A
- new net A5: LED5.A
- new net A6: LED6.A
- new net A7: LED7.A
- new net A8: LED8.A
- new net B1: LED1.A
- new net B2: LED2.A
- new net B3: LED3.A
- new net B4: LED4.A
- new net B5: LED5.A
- new net B6: LED6.A
- new net B7: LED7.A
- new net B8: LED8.A
- new net CLK_HLT: R7.2
- new net CLK_OUT: LED1.A
- new net D1: LED1.A, R1.2
- new net D2: LED2.A, R2.2
- new net D3: LED3.A, R3.2
- new net D4: LED4.A, R4.2
- new net D5: LED5.A, R5.2
- new net D6: LED6.A, R6.2
- new net D7: LED7.A, R7.2
- new net D8: LED8.A, R8.2
- new net GND: LED1.C, LED2.C, LED3.C, LED4.C, LED5.C, LED6.C, LED7.C, LED8.C, R1.1, R1.2, R2.1, R2.2, R3.1, R3.2, R4.1, R4.2, R5.1, R5.2, R6.1, R6.2, R7.1, R7.2, R8.1, R8.2
- new net I1: LED1.A
- new net I2: LED2.A
- new net I3: LED3.A
- new net I4: LED4.A
- new net I5: LED5.A
- new net I6: LED6.A
- new net I7: LED7.A
- new net I8: LED8.A
- new net N$1: R2.A, R2.S
- new net N$10: LED2.C, R2.1
- new net N$11: LED3.C, R3.1, R5.1
- new net N$12: LED4.C, R4.1
- new net N$13: LED5.C, R1.1, R3.2, R5.1
- new net N$14: LED6.C, R6.1
- new net N$15: LED7.C, R7.1
- new net N$16: LED8.C, R3.1, R8.1
- new net N$2: LED2.C, R1.1, R2.1, R3.2
- new net N$3: LED3.C, R2.E, R3.1
- new net N$4: LED1.C, LED4.C, R1.1, R4.1, R4.2
- new net N$5: LED5.C, R5.1
- new net N$6: LED6.C, R6.1
- new net N$7: LED7.C, R6.1, R7.1
- new net N$8: LED8.C, R8.1
- new net N$9: LED1.C, R1.1
- new net Q1: LED1.A
- new net Q2: LED2.A
- new net Q3: LED3.A
- new net Q4: LED4.A
- new net S1: LED1.A
- new net S2: LED2.A
- new net S3: LED3.A
- new net S4: LED4.A
- new net S5: LED5.A
- new net S6: LED6.A
- new net S7: LED7.A
- new net S8: LED8.A
- new net VCC: R1.2, R5.2, R6.2

Commit message: added instruction decoder module
Parts:
- added R10, R11, R12, R13, R14, R15, R16, R9: 470, rcl:R-US_0204/7
Connections:
- new net !AI: LED8.A
- new net !AO: LED7.A
- new net !II: LED6.A
- new net !IO: LED5.A
- new net !MI: LED2.A
- new net !RO: LED3.A
- new net HLT: LED1.A
- new net N$23: LED1.A, R9.1
- new net N$24: LED2.A, R10.1
- new net N$25: LED3.A, R11.1
- new net N$26: LED4.A, R12.1
- new net N$27: LED5.A, R13.1, R9.2
- new net N$28: LED6.A, R14.1
- new net N$29: LED7.A, R15.1
- new net N$30: LED8.A, R16.1
- new net P/R: R9.2
- new net RI: LED4.A
- net D1: now also R9.2; no longer LED1.A
- net D2: now also R10.2; no longer LED2.A
- net D3: now also R11.2; no longer LED3.A
- net D4: now also R12.2; no longer LED4.A
- net D5: now also R13.2; no longer LED5.A
- net D6: now also R14.2; no longer LED6.A
- net D7: now also R15.2; no longer LED7.A
- net D8: now also R16.2; no longer LED8.A
- net GND: now also R10.1, R11.1, R12.1, R13.1, R14.1, R15.1, R16.1, R9.1; no longer R1.2, R2.2, R3.2, R4.2, R5.2, R6.2, R7.2, R8.2
- net N$1: now also LED1.C, R1.2
- net N$10: now also R10.2; no longer LED2.C, R2.1
- net N$11: now also R11.2; no longer LED3.C, R3.1
- net N$12: now also R12.2; no longer LED4.C, R4.1
- net N$13: now also R10.1, R13.2; no longer LED5.C, R5.1
- net N$14: now also R14.2; no longer LED6.C, R6.1
- net N$15: now also R15.2, R9.1; no longer LED7.C, R7.1
- net N$16: now also LED1.C, LED2.C, LED3.C, LED4.C, LED5.C, LED6.C, LED7.C, R10.1, R16.2; no longer R8.1
- net N$2: now also R2.2; no longer R2.1
- net N$3: now also R3.2
- net N$4: now also LED2.C, LED3.C, LED5.C, LED6.C, LED7.C, LED8.C; no longer R1.1, R4.1
- net N$5: now also R5.2; no longer R5.1
- net N$6: now also R6.2; no longer R6.1
- net N$7: now also R10.2, R7.2; no longer R7.1
- net N$8: now also R8.2; no longer R8.1
- net N$9: now also LED2.C, LED3.C, LED4.C, LED5.C, LED6.C, LED7.C, LED8.C, R9.1, R9.2; no longer R1.1
- net VCC: now also R10.2, R9.2
Other:
- note added: "Control Word Output"
- note added: "Instruction Decoder & Control Logic"
- note added: "Microinstruction Counter w/ 5 Steps"
- note added: "Reset Button"
- moved on the sheet: LED1, LED2, LED3, LED4, LED5, LED6, LED7, LED8

Commit message: added CPU status register
Connections:
- net !MI renamed CF
- net HLT renamed ZF
- removed net !AI: LED8.A
- removed net !AO: LED7.A
- removed net !II: LED6.A
- removed net !IO: LED5.A
- removed net !RO: LED3.A
- removed net RI: LED4.A
- new net N$31: R16.2
- net N$1: no longer LED1.C
- net N$16: no longer LED1.C, LED2.C, LED3.C, LED4.C, LED5.C, LED6.C, LED7.C, LED8.C, R16.2
- net N$2: no longer LED2.C
- net N$3: no longer LED3.C
- net N$5: no longer LED5.C
- net N$6: no longer LED6.C
- net N$7: no longer LED7.C
- net N$8: no longer LED8.C
- net N$9: no longer LED1.C, LED2.C, LED3.C, LED4.C, LED5.C, LED6.C, LED7.C, LED8.C
Other:
- note added: "1st Byte in Control Word Base Address: 0x00"
- note added: "2nd Byte in Control Word Base Address: 0x80"
- note added: "8-bit Adder w/ 2's Substract"
- note added: "Zero Detect"
- moved on the sheet: LED1, LED2, LED3, LED4, LED5, LED6, LED7, LED8, R10, R11, R12, R13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

Commit message: added current limiting resistors
Parts:
- R10, R11, R12, R13, R14, R15, R16, R9: value 470 -> 220; MOUSER 594-5063JD1K000F -> 594-5063JD220R0F
Connections:
- removed net CLK_HLT: R7.2
- net N$1: now also LED1.C, LED4.C, LED8.C, R2.2, R4.2, R8.2
- net N$10: now also LED1.C, LED6.C, LED7.C, R1.2, R6.2, R7.2
- net N$11: now also LED5.C, LED6.C, R5.2, R6.2
- net N$12: now also LED4.C, LED5.C, R4.2, R5.2
- net N$13: now also LED3.C, LED4.C, R4.2
- net N$14: now also LED2.C, LED3.C, R2.2, R3.2
- net N$15: now also LED1.C, LED2.C, R1.2, R2.2
- net N$16: now also LED1.C, R1.2
- net N$2: now also LED2.C, LED3.C, LED4.C, LED7.C, R1.2, R4.2, R7.2
- net N$3: now also LED2.C, LED3.C, LED6.C, R2.2, R6.2
- net N$4: now also R1.1, R1.2, R11.2, R2.1, R3.1, R3.2, R4.1, R5.1, R5.2, R6.1, R7.1, R8.1; no longer LED2.C, LED6.C, LED7.C, LED8.C
- net N$5: now also LED4.C, LED5.C, R4.2
- net N$6: now also LED3.C, LED4.C, LED6.C, R3.2, R4.2
- net N$7: now also LED2.C, LED3.C, LED7.C, R2.2, R3.2
- net N$8: now also LED1.C, LED2.C, LED8.C, R1.2, R2.2
- net N$9: now also LED1.C, LED7.C, LED8.C, R1.2, R7.2, R8.2

Commit message: added mouser part numbers
Parts:
- LED1, LED2, LED3, LED4, LED5, LED6, LED7, LED8: value (none) -> RED; MOUSER 941-C503BRANCZ0C0AA1 -> 743-INL-3AR30
- R1, R2, R3, R4, R5, R6, R7, R8: MOUSER 594-5063JD1K000F -> 594-5063JD10K00F
