File: Board/SAP-1.sch (EAGLE design)
At the start: 24 parts

Commit message: added BOM
Parts:
- added C1: (no value), rcl:CPOL-EUE3.5-8
- added C6: 100n, rcl:C-EU050-024X044
- added U$1: DC-JACK, Parts:DC-JACK
Connections:
- net GND: now also C1.-, C1.2, C6.2, U$1.GND, U$1.GNDBREAK
- net N$1: now also C1.+
- net VCC: now also C1.+, C1.1, C6.1, U$1.PWR
Changed lines of the file:
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@@
 <layer number="112" name="tSilk" color="7" fill="1" visible="yes" active="yes"/>
 <layer number="113" name="IDFDebug" color="7" fill="1" visible="yes" active="yes"/>
+<layer number="114" name="Badge_Outline" color="7" fill="1" visible="yes" active="yes"/>
+<layer number="115" name="ReferenceISLANDS" color="7" fill="1" visible="yes" active="yes"/>
 <layer number="116" name="Patch_BOT" color="9" fill="4" visible="yes" active="yes"/>
+<layer number="117" name="BACKMAAT1" color="7" fill="1" visible="yes" active="yes"/>
 <layer number="118" name="Rect_Pads" color="7" fill="1" visible="yes" active="yes"/>
+<layer number="119" name="KAP_TEKEN" color="7" fill="1" visible="yes" active="yes"/>
+<layer number="120" name="KAP_MAAT1" color="7" fill="1" visible="yes" active="yes"/>
 <layer number="121" name="_tsilk" color="7" fill="1" visible="yes" active="yes"/>
 <layer number="122" name="_bsilk" color="7" fill="1" visible="yes" active="yes"/>
@@
 <layer number="128" name="_bValues" color="7" fill="1" visible="yes" active="yes"/>
 <layer number="129" name="Mask" color="7" fill="1" visible="yes" active="yes"/>
+<layer number="130" name="SMDSTROOK" color="7" fill="1" visible="yes" active="yes"/>
 <layer number="131" name="tAdjust" color="7" fill="1" visible="yes" active="yes"/>
 <layer number="132" name="bAdjust" color="7" fill="1" visible="yes" active="yes"/>
+<layer number="133" name="bottom_silk" color="7" fill="1" visible="yes" active="yes"/>
+<layer number="134" name="silk_top" color="7" fill="1" visible="no" active="no"/>
+<layer number="135" name="silk_bottom" color="7" fill="1" visible="no" active="no"/>
+<layer number="136" name="silktop" color="7" fill="1" visible="yes" active="yes"/>
+<layer number="137" name="silkbottom" color="7" fill="1" visible="yes" active="yes"/>
 <layer number="144" name="Drill_legend" color="7" fill="1" visible="yes" active="yes"/>
+<layer number="145" name="DrillLegend_01-16" color="7" fill="1" visible="yes" active="yes"/>
+<layer number="146" name="DrillLegend_01-20" color="7" fill="1" visible="yes" active="yes"/>
 <layer number="150" name="Notes" color="7" fill="1" visible="yes" active="yes"/>
 <layer number="151" name="HeatSink" color="7" fill="1" visible="yes" active="yes"/>
@@
 <layer number="230" name="230bmp" color="7" fill="1" visible="yes" active="yes"/>
 <layer number="231" name="231bmp" color="7" fill="1" visible="yes" active="yes"/>
+<layer number="232" name="Eagle3D_PG2" color="7" fill="1" visible="yes" active="yes"/>
+<layer number="233" name="Eagle3D_PG3" color="7" fill="1" visible="yes" active="yes"/>
 <layer number="248" name="Housing" color="7" fill="1" visible="yes" active="yes"/>
 <layer number="249" name="Edge" color="7" fill="1" visible="yes" active="yes"/>
@@
 </pinmapping>
 </spice>
-<attribute name="CONRAD" value="445639"/>
 <attribute name="MOUSER" value="710-860021373002"/>
 </part>
@@
 <attribute name="NAME" x="17.907" y="19.083" size="1.778" layer="95"/>
 <attribute name="VALUE" x="17.907" y="15.0368" size="1.778" layer="96" align="top-left"/>
-<attribute name="CONRAD" x="15.24" y="17.78" size="1.778" layer="96" display="off"/>
 <attribute name="MOUSER" x="15.24" y="17.78" size="1.778" layer="96" display="off"/>
 </instance>
@@
 <attribute name="MOUSER" value="594-5063JD220R0F"/>
 </part>
+<part name="C1" library="rcl" library_urn="urn:adsk.eagle:library:334" deviceset="CPOL-EU" device="E3.5-8" package3d_urn="urn:adsk.eagle:package:23360/2">
+<spice>
+<pinmapping spiceprefix="C">
+<pinmap gate="G$1" pin="+" pinorder="1"/>
+<pinmap gate="G$1" pin="-" pinorder="2"/>
+</pinmapping>
+</spice>
+<attribute name="MOUSER" value="710-860040674004"/>
+</part>
+<part name="U$1" library="Parts" library_urn="urn:adsk.eagle:library:2304016" deviceset="DC-JACK" device="" package3d_urn="urn:adsk.eagle:package:2338719/2"/>
+<part name="C6" library="rcl" library_urn="urn:adsk.eagle:library:334" deviceset="C-EU" device="050-024X044" package3d_urn="urn:adsk.eagle:package:23643/1" value="100n">
+<spice>
+<pinmapping spiceprefix="C">
+<pinmap gate="G$1" pin="1" pinorder="1"/>
+<pinmap gate="G$1" pin="2" pinorder="2"/>
+</pinmapping>
+</spice>
+<attribute name="MOUSER" value="594-K104K15X7RF53H5"/>
+</part>
+<part name="GND5" library="supply1" library_urn="urn:adsk.eagle:library:371" deviceset="GND" device=""/>
+<part name="P+8" library="supply1" library_urn="urn:adsk.eagle:library:371" deviceset="VCC" device=""/>
 </parts>
 <sheets>
@@
 <attribute name="MOUSER" x="53.34" y="-111.76" size="1.778" layer="96" rot="R90" display="off"/>
 </instance>
+<instance part="C1" gate="G$1" x="15.24" y="157.48" smashed="yes">
+<attribute name="NAME" x="16.383" y="157.9626" size="1.778" layer="95"/>
+<attribute name="VALUE" x="16.383" y="152.8826" size="1.778" layer="96"/>
+<attribute name="MOUSER" x="15.24" y="157.48" size="1.778" layer="96" display="off"/>
+</instance>
+<instance part="U$1" gate="G$1" x="5.08" y="152.4" smashed="yes">
+<attribute name="VALUE" x="-5.08" y="162.56" size="1.778" layer="96" font="vector"/>
+<attribute name="NAME" x="-5.08" y="152.4" size="1.778" layer="95" font="vector"/>
+</instance>
+<instance part="C6" gate="G$1" x="22.86" y="157.48" smashed="yes">
+<attribute name="NAME" x="24.892" y="157.6832" size="1.778" layer="95"/>
+<attribute name="VALUE" x="24.892" y="154.7368" size="1.778" layer="96" align="top-left"/>
+<attribute name="MOUSER" x="22.86" y="157.48" size="1.778" layer="96" display="off"/>
+</instance>
+<instance part="GND5" gate="1" x="15.24" y="147.32" smashed="yes">
+<attribute name="VALUE" x="12.7" y="144.78" size="1.778" layer="96"/>
+</instance>
+<instance part="P+8" gate="VCC" x="15.24" y="165.1" smashed="yes">
+<attribute name="VALUE" x="12.7" y="162.56" size="1.778" layer="96" rot="R90"/>
+</instance>
 </instances>
 <busses>
@@
 <junction x="83.82" y="-129.54"/>
 </segment>
+<segment>
+<pinref part="U$1" gate="G$1" pin="GNDBREAK"/>
+<pinref part="U$1" gate="G$1" pin="GND"/>
+<wire x1="7.62" y1="157.48" x2="7.62" y2="154.94" width="0.1524" layer="91"/>
+<wire x1="7.62" y1="154.94" x2="7.62" y2="152.4" width="0.1524" layer="91"/>
+<junction x="7.62" y="154.94"/>
+<pinref part="C1" gate="G$1" pin="-"/>
+<wire x1="7.62" y1="152.4" x2="15.24" y2="152.4" width="0.1524" layer="91"/>
+<pinref part="C6" gate="G$1" pin="2"/>
+<wire x1="15.24" y1="152.4" x2="22.86" y2="152.4" width="0.1524" layer="91"/>
+<junction x="15.24" y="152.4"/>
+<pinref part="GND5" gate="1" pin="GND"/>
+<wire x1="15.24" y1="149.86" x2="15.24" y2="152.4" width="0.1524" layer="91"/>
+</segment>
 </net>
 <net name="N$22" class="0">
@@
 </segment>
 </net>
+<net name="VCC" class="0">
+<segment>
+<pinref part="U$1" gate="G$1" pin="PWR"/>
+<pinref part="C1" gate="G$1" pin="+"/>
+<wire x1="7.62" y1="160.02" x2="15.24" y2="160.02" width="0.1524" layer="91"/>
+<pinref part="C6" gate="G$1" pin="1"/>
+<wire x1="22.86" y1="160.02" x2="15.24" y2="160.02" width="0.1524" layer="91"/>
+<junction x="15.24" y="160.02"/>
+<pinref part="P+8" gate="VCC" pin="VCC"/>
+<wire x1="15.24" y1="160.02" x2="15.24" y2="162.56" width="0.1524" layer="91"/>
+</segment>
+</net>

Commit message: layed out components on board
Connections:
- new net N$17: R12.2
- new net SEG_A: R8.1
- new net SEG_AO: R8.2
- new net SEG_B: R9.1
- new net SEG_BO: R9.2
- new net SEG_C: R10.1
- new net SEG_CO: R10.2
- new net SEG_D: R11.1
- new net SEG_DO: R11.2
- new net SEG_DP: R15.1
- new net SEG_DPO: R15.2
- new net SEG_E: R12.1
- new net SEG_F: R13.1
- new net SEG_FO: R13.2
- new net SEG_G: R14.1
- new net SEG_GO: R14.2

Commit message: replace most discrete resistors with networks
Parts:
- removed R1, R2, R3, R4, R5, R6, R7, R8: 10k, rcl:R-US_0204/7
- removed R10, R11, R12, R13, R14, R15, R16, R9: 220, rcl:R-US_0204/7
- added RN1: 10k, resistor-sil:GE08R
- added RN3: 220, resistor-sil:GE08R
- C1: value (none) -> 100u
Connections:
- removed net N$17: R12.2
- removed net N$31: R16.2
- removed net P/R: R9.2
- removed net SEG_C: R10.1
- removed net SEG_CO: R10.2
- removed net SEG_D: R11.1
- removed net SEG_DO: R11.2
- removed net SEG_DP: R15.1
- removed net SEG_DPO: R15.2
- removed net SEG_E: R12.1
- new net N$33: RN3C.2
- new net N$34: RN3A.2
- new net N$35: RN3B.2
- new net N$36: RN3D.2
- new net N$37: RN3E.2
- net D1: now also LED1.A, RN1H.2; no longer R1.2, R9.2
- net D2: now also LED2.A, RN1G.2; no longer R10.2, R2.2
- net D3: now also LED3.A, RN1F.2; no longer R11.2, R3.2
- net D4: now also LED4.A, RN1E.2; no longer R12.2, R4.2
- net D5: now also LED5.A, RN1D.2; no longer R13.2, R5.2
- net D6: now also LED6.A, RN1C.2; no longer R14.2, R6.2
- net D7: now also LED7.A, RN1B.2; no longer R15.2, R7.2
- net D8: now also LED8.A, RN1A.2; no longer R16.2, R8.2
- net GND: now also RN1A.1, RN3A.1; no longer LED1.C, LED2.C, LED3.C, LED4.C, LED5.C, LED6.C, LED7.C, LED8.C, R1.1, R10.1, R11.1, R12.1, R13.1, R14.1, R15.1, R16.1, R2.1, R3.1, R4.1, R5.1, R6.1, R7.1, R8.1, R9.1
- net N$1: now also RN1A.2, RN1D.2, RN3A.2, RN3H.2; no longer R1.2, R2.2, R2.A, R2.S, R4.2, R8.2
- net N$10: now also RN1A.2, RN3F.2, RN3G.2; no longer R1.2, R10.2, R6.2, R7.2
- net N$11: now also RN3E.2, RN3F.2; no longer R11.2, R5.1, R5.2, R6.2
- net N$12: now also RN3D.2, RN3E.2; no longer R12.2, R4.2, R5.2
- net N$13: now also RN3C.2, RN3D.2; no longer R1.1, R10.1, R13.2, R3.2, R4.2
- net N$14: now also RN3B.2, RN3C.2; no longer R14.2, R2.2, R3.2
- net N$15: now also RN3A.2, RN3B.2; no longer R1.2, R15.2, R2.2, R9.1
- net N$16: now also RN3A.2; no longer R1.2, R10.1, R3.1
- net N$2: now also RN1B.2, RN1C.2, RN1D.2, RN3B.2, RN3G.2; no longer R1.1, R1.2, R2.2, R3.2, R4.2, R7.2
- net N$23: now also LED8.C, RN3A.2; no longer LED1.A, R9.1
- net N$24: now also LED7.C, RN3B.2; no longer LED2.A, R10.1
- net N$25: now also LED6.C, RN3C.2; no longer LED3.A, R11.1
- net N$26: now also LED5.C, RN3D.2; no longer LED4.A, R12.1
- net N$27: now also LED4.C, RN3E.2; no longer LED5.A, R13.1, R9.2
- net N$28: now also LED3.C, RN3F.2; no longer LED6.A, R14.1
- net N$29: now also LED2.C, RN3G.2; no longer LED7.A, R15.1
- net N$3: now also RN1B.2, RN1C.2, RN3C.2, RN3F.2; no longer R2.2, R2.E, R3.1, R3.2, R6.2
- net N$30: now also LED1.C, RN3H.2; no longer LED8.A, R16.1
- net N$4: now also RN1A.2, RN1C.2, RN1D.2, RN3D.2, RN3E.2; no longer R1.1, R1.2, R11.2, R2.1, R3.1, R3.2, R4.1, R4.2, R5.1, R5.2, R6.1, R7.1, R8.1
- net N$5: now also RN1E.2, RN3D.2, RN3E.2; no longer R4.2, R5.2
- net N$6: now also RN1F.2, RN3C.2, RN3D.2, RN3F.2; no longer R3.2, R4.2, R6.2
- net N$7: now also RN1G.2, RN3B.2, RN3C.2, RN3G.2; no longer R10.2, R2.2, R3.2, R6.1, R7.2
- net N$8: now also RN1B.2, RN1H.2, RN3A.2, RN3B.2, RN3H.2; no longer R1.2, R2.2, R8.2
- net N$9: now also RN3A.2, RN3G.2, RN3H.2; no longer R1.2, R7.2, R8.2, R9.1, R9.2
- net SEG_A: now also RN1C.2; no longer R8.1
- net SEG_AO: now also RN1C.1; no longer R8.2
- net SEG_B: now also RN1D.2; no longer R9.1
- net SEG_BO: now also RN1D.1; no longer R9.2
- net SEG_F: now also RN1B.2; no longer R13.1
- net SEG_FO: now also RN1B.1; no longer R13.2
- net SEG_G: now also RN1A.2; no longer R14.1
- net SEG_GO: now also RN1A.1; no longer R14.2
- net VCC: no longer R1.2, R10.2, R5.2, R6.2, R9.2
Other:
- moved on the sheet: LED1, LED2, LED3, LED4, LED5, LED6, LED7, LED8

Commit message: started routing of modules
Connections:
- new net N$18: RN1H.2
- new net N$19: RN1G.2
- new net N$20: RN1F.2
- new net N$21: RN1E.2
- new net N$22: RN1D.2
- net N$23: now also RN1C.2
- net N$24: now also RN1B.2
- net N$25: now also RN1A.2
- net VCC: now also RN1A.1

Commit message: added mounting holes
Parts:
- added H1, H2, H3, H4, H5, H6: MOUNT-PAD-ROUND3.2, holes:MOUNT-PAD-ROUND3.2
Connections:
- net GND: now also H1.MOUNT, H2.MOUNT, H3.MOUNT, H4.MOUNT, H5.MOUNT, H6.MOUNT
Changed lines of the file:
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@@
 <part name="P+11" library="supply1" library_urn="urn:adsk.eagle:library:371" deviceset="VCC" device=""/>
 <part name="P+12" library="supply1" library_urn="urn:adsk.eagle:library:371" deviceset="VCC" device=""/>
+<part name="H1" library="holes" library_urn="urn:adsk.eagle:library:237" deviceset="MOUNT-PAD-ROUND" device="3.2" package3d_urn="urn:adsk.eagle:package:14282/1"/>
+<part name="H2" library="holes" library_urn="urn:adsk.eagle:library:237" deviceset="MOUNT-PAD-ROUND" device="3.2" package3d_urn="urn:adsk.eagle:package:14282/1"/>
+<part name="H3" library="holes" library_urn="urn:adsk.eagle:library:237" deviceset="MOUNT-PAD-ROUND" device="3.2" package3d_urn="urn:adsk.eagle:package:14282/1"/>
+<part name="H4" library="holes" library_urn="urn:adsk.eagle:library:237" deviceset="MOUNT-PAD-ROUND" device="3.2" package3d_urn="urn:adsk.eagle:package:14282/1"/>
+<part name="GND15" library="supply1" library_urn="urn:adsk.eagle:library:371" deviceset="GND" device=""/>
+<part name="H5" library="holes" library_urn="urn:adsk.eagle:library:237" deviceset="MOUNT-PAD-ROUND" device="3.2" package3d_urn="urn:adsk.eagle:package:14282/1"/>
+<part name="H6" library="holes" library_urn="urn:adsk.eagle:library:237" deviceset="MOUNT-PAD-ROUND" device="3.2" package3d_urn="urn:adsk.eagle:package:14282/1"/>
 </parts>
 <sheets>
@@
 <attribute name="VALUE" x="134.62" y="127" size="1.778" layer="96" rot="R90"/>
 </instance>
+<instance part="H1" gate="G$1" x="38.1" y="160.02" smashed="yes" rot="R180">
+<attribute name="NAME" x="35.306" y="159.4358" size="1.778" layer="95" rot="R180"/>
+<attribute name="VALUE" x="35.306" y="162.4838" size="1.778" layer="96" rot="R180"/>
+</instance>
+<instance part="H2" gate="G$1" x="48.26" y="160.02" smashed="yes">
+<attribute name="NAME" x="51.054" y="160.6042" size="1.778" layer="95"/>
+<attribute name="VALUE" x="51.054" y="157.5562" size="1.778" layer="96"/>
+</instance>
+<instance part="H3" gate="G$1" x="48.26" y="152.4" smashed="yes">
+<attribute name="NAME" x="51.054" y="152.9842" size="1.778" layer="95"/>
+<attribute name="VALUE" x="51.054" y="149.9362" size="1.778" layer="96"/>
+</instance>
+<instance part="H4" gate="G$1" x="38.1" y="152.4" smashed="yes" rot="R180">
+<attribute name="NAME" x="35.306" y="151.8158" size="1.778" layer="95" rot="R180"/>
+<attribute name="VALUE" x="35.306" y="154.8638" size="1.778" layer="96" rot="R180"/>
+</instance>
+<instance part="GND15" gate="1" x="43.18" y="147.32" smashed="yes">
+<attribute name="VALUE" x="40.64" y="144.78" size="1.778" layer="96"/>
+</instance>
+<instance part="H5" gate="G$1" x="38.1" y="167.64" smashed="yes" rot="R180">
+<attribute name="NAME" x="35.306" y="167.0558" size="1.778" layer="95" rot="R180"/>
+<attribute name="VALUE" x="35.306" y="170.1038" size="1.778" layer="96" rot="R180"/>
+</instance>
+<instance part="H6" gate="G$1" x="48.26" y="167.64" smashed="yes">
+<attribute name="NAME" x="51.054" y="168.2242" size="1.778" layer="95"/>
+<attribute name="VALUE" x="51.054" y="165.1762" size="1.778" layer="96"/>
+</instance>
 </instances>
 <busses>
@@
 <wire x1="-2.54" y1="101.6" x2="-2.54" y2="99.06" width="0.1524" layer="91"/>
 </segment>
-</net>
+<segment>
+<pinref part="H1" gate="G$1" pin="MOUNT"/>
+<pinref part="H2" gate="G$1" pin="MOUNT"/>
+<wire x1="40.64" y1="160.02" x2="43.18" y2="160.02" width="0.1524" layer="91"/>
+<pinref part="H3" gate="G$1" pin="MOUNT"/>
+<pinref part="H4" gate="G$1" pin="MOUNT"/>
+<wire x1="43.18" y1="160.02" x2="45.72" y2="160.02" width="0.1524" layer="91"/>
+<wire x1="45.72" y1="152.4" x2="43.18" y2="152.4" width="0.1524" layer="91"/>
+<wire x1="43.18" y1="152.4" x2="40.64" y2="152.4" width="0.1524" layer="91"/>
+<wire x1="43.18" y1="160.02" x2="43.18" y2="152.4" width="0.1524" layer="91"/>
+<junction x="43.18" y="160.02"/>
+<junction x="43.18" y="152.4"/>
+<pinref part="GND15" gate="1" pin="GND"/>
+<wire x1="43.18" y1="149.86" x2="43.18" y2="152.4" width="0.1524" layer="91"/>
+<pinref part="H5" gate="G$1" pin="MOUNT"/>
+<pinref part="H6" gate="G$1" pin="MOUNT"/>
+<wire x1="40.64" y1="167.64" x2="43.18" y2="167.64" width="0.1524" layer="91"/>
+<wire x1="43.18" y1="167.64" x2="45.72" y2="167.64" width="0.1524" layer="91"/>
+<wire x1="43.18" y1="160.02" x2="43.18" y2="167.64" width="0.1524" layer="91"/>
+<junction x="43.18" y="167.64"/>
+</segment>
+</net>
