File: Board/SAP-1.sch (EAGLE design)
At the start: 19 parts

Commit message: Second Silkscreen cleanup pass
Parts:
- added TP1, TP2, TP3, TP4, TP5, TP6, TP7, TP8: TPTP06R, testpad:TPTP06R
Connections:
- new net !AI: TP8.TP
- new net !AO: TP7.TP
- new net !CLK_OUT: TP1.TP
- new net !II: TP6.TP
- new net !IO: TP5.TP
- new net !MI: TP2.TP
- new net !RO: TP3.TP
- new net CY: TP1.TP
- new net HLT: TP1.TP
- new net RI: TP4.TP
- new net ZR: TP2.TP
- net CLK_OUT: now also TP2.TP
- net D1: now also TP8.TP
- net D2: now also TP7.TP
- net D3: now also TP6.TP
- net D4: now also TP5.TP
- net D5: now also TP4.TP
- net D6: now also TP3.TP
- net D7: now also TP2.TP
- net D8: now also TP1.TP
Other:
- note added: "Unused Gates"
- note added: "Unused Gatres"

Commit message: updated attributes of resistor networks
Parts:
- added J1, J2: TERMINAL-1BRIDGE, AdapterBoard:TERMINAL-1BRIDGE
- added TP10, TP11, TP12, TP13, TP14, TP15, TP16, TP9: TPTP06R, testpad:TPTP06R
- H5, H6: value MOUNT-PAD-ROUND3.2 -> 3.2
Connections:
- new net !BI: TP11.TP
- new net !CO: TP14.TP
- new net !EO: TP9.TP
- new net !FI: TP16.TP
- new net !JP: TP15.TP
- new net CE: TP13.TP
- new net OI: TP12.TP
- new net SU: TP10.TP
- net !CLK_OUT: now also TP4.TP
- net CLK_OUT: now also TP3.TP
- net CY: now also TP4.TP
- net D1: now also TP16.TP
- net D2: now also TP15.TP
- net D3: now also TP14.TP
- net D4: now also TP13.TP
- net D5: now also TP12.TP
- net D6: now also TP11.TP
- net D7: now also TP10.TP
- net D8: now also TP9.TP
- net GND: now also J2.P$1
- net VCC: now also J1.P$1
- net ZR: now also TP3.TP

Commit message: removed buffering of instruction register upper nibble
Connections:
- net I1: now also LED5.A
- net I2: now also LED6.A
- net I3: now also LED7.A
- net I4: now also LED8.A
